File: SDCard.kicad_sch (KiCad schematic)
At the start: 1 part, among them J9 Micro_SD_Card

Commit message: Beginnings of routing
Parts:
- J9: footprint Connector_Card:microSD_HC_Molex_47219-2001 -> Connector_Card:microSD_HC_Hirose_DM3D-SF
Changed lines of the file:
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@@
 		(dnp no)
 		(fields_autoplaced yes)
-		(property "Reference" "#PWR0105"
+		(property "Reference" "#PWR0110"
 			(at 123.19 86.36 0)
 			(effects
@@
 			(project "Cubesat-FC-V1"
 				(path "/f01d9098-91c1-4e97-a02a-fecce6a76317/ca6c8c54-a6c6-4650-9150-e5152dbc00db"
-					(reference "#PWR0105")
+					(reference "#PWR0110")
 					(unit 1)
 				)
@@
 		(dnp no)
 		(fields_autoplaced yes)
-		(property "Reference" "#PWR0104"
+		(property "Reference" "#PWR0109"
 			(at 67.31 76.2 0)
 			(effects
@@
 			(project ""
 				(path "/f01d9098-91c1-4e97-a02a-fecce6a76317/ca6c8c54-a6c6-4650-9150-e5152dbc00db"
-					(reference "#PWR0104")
+					(reference "#PWR0109")
 					(unit 1)
 				)
@@
 			)
 		)
-		(property "Footprint" "Connector_Card:microSD_HC_Molex_47219-2001"
+		(property "Footprint" "Connector_Card:microSD_HC_Hirose_DM3D-SF"
 			(at 130.81 55.88 0)
 			(effects
@@
 		(dnp no)
 		(fields_autoplaced yes)
-		(property "Reference" "#PWR0103"
+		(property "Reference" "#PWR0108"
 			(at 67.31 66.04 0)
 			(effects
@@
 			(project ""
 				(path "/f01d9098-91c1-4e97-a02a-fecce6a76317/ca6c8c54-a6c6-4650-9150-e5152dbc00db"
-					(reference "#PWR0103")
-					(unit 1)
-				)
+					(reference "#PWR0108")
+					(unit 1)
+				)

Commit message: Formatting
Other:
- company: (none) -> UMASS Cubesat Lab
Changed lines of the file:
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@@
 	(generator_version "9.0")
 	(paper "A5")
+	(title_block
+		(date "2026-03-22")
+		(rev "R1")
+		(company "UMASS Cubesat Lab")
+	)
 	(wire
 		(pts
