File: SDRAM.kicad_sch (KiCad schematic)
At the start: 1 part

Commit message: Finish IMS, finished more work on schematic
Parts:
- added C49: 1u, Capacitor_SMD:C_0402_1005Metric, symbol Device:C_Small
- added C50: 0.1u, Capacitor_SMD:C_0402_1005Metric, symbol Device:C_Small
- renumbered U2 to U4
Connections:
- net +3.3V: now reaches U4.1 (VDD), U4.14 (VDD), U4.27 (VDD)
- net +3.3V: now also U4.3 (VDDQ), U4.43 (VDDQ), U4.49 (VDDQ), U4.9 (VDDQ), C49.1, C50.1
- net GND: now reaches U4.12 (VSSQ), U4.46 (VSSQ), U4.52 (VSSQ), U4.6 (VSSQ)
- net GND: now also U4.28 (VSS), U4.41 (VSS), U4.54 (VSS), C49.2, C50.2
- no-connect marks 0 -> 1
Other:
- moved on the sheet: U4

Commit message: Beginnings of routing
Parts:
- renumbered U4 to U5
Changed lines of the file:
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@@
-	(bus
-		(pts
-			(xy 31.75 20.32) (xy 54.61 20.32)
-		)
-		(stroke
-			(width 0)
-			(type default)
-		)
-	)
 	(bus
 		(pts
@@
 		)
 	)
-	(label "FMC{A[0..12] D[0..15]}"
-		(at 31.75 20.32 0)
-		(effects
-			(font
-				(size 1.27 1.27)
-			)
-			(justify left bottom)
-		)
-	)
 	(label "FMCD9"
 		(at 118.11 49.53 180)
@@
 		)
 	)
-	(label "FMC{A[0..12] D[0..15]}"
-		(at 144.78 24.13 180)
-		(effects
-			(font
-				(size 1.27 1.27)
-			)
-			(justify right bottom)
-		)
-	)
 	(label "FMCA5"
 		(at 72.39 44.45 0)
@@
 		)
 	)
-	(label "FMC{A[0..12] D[0..15]}"
-		(at 45.72 64.77 0)
-		(effects
-			(font
-				(size 1.27 1.27)
-			)
-			(justify left bottom)
-		)
-	)
 	(label "FMCD1"
 		(at 118.11 29.21 180)
@@
 			)
 			(justify right bottom)
-		)
-	)
-	(hierarchical_label "FMC{A[0..12] D[0..15]}"
-		(shape input)
-		(at 54.61 20.32 0)
-		(effects
-			(font
-				(size 1.27 1.27)
-			)
-			(justify left)
 		)
 	)
@@
 			)
 			(justify right)
+		)
+	)
+	(hierarchical_label "FMCA[0..12]"
+		(shape input)
+		(at 45.72 64.77 180)
+		(effects
+			(font
+				(size 1.27 1.27)
+			)
+			(justify right)
+		)
+	)
+	(hierarchical_label "FMCD[0..15]"
+		(shape input)
+		(at 144.78 24.13 0)
+		(effects
+			(font
+				(size 1.27 1.27)
+			)
+			(justify left)
 		)
 	)
@@
 		(dnp no)
 		(fields_autoplaced yes)
-		(property "Reference" "U4"
+		(property "Reference" "U5"
 			(at 98.6633 20.32 0)
 			(effects
@@
 			(project "Cubesat-FC-V1"
 				(path "/f01d9098-91c1-4e97-a02a-fecce6a76317/353c0638-7d15-4c84-b70a-670532d5bdf1"
-					(reference "U4")
+					(reference "U5")
 					(unit 1)
 				)
@@
 		(on_board yes)
 		(dnp no)
-		(property "Reference" "#PWR063"
+		(property "Reference" "#PWR068"
 			(at 93.98 22.86 0)
 			(effects
@@
 			(project ""
 				(path "/f01d9098-91c1-4e97-a02a-fecce6a76317/353c0638-7d15-4c84-b70a-670532d5bdf1"
-					(reference "#PWR063")
+					(reference "#PWR068")
 					(unit 1)
 				)
@@
 		(dnp no)
 		(fields_autoplaced yes)
-		(property "Reference" "#PWR066"
+		(property "Reference" "#PWR070"
 			(at 139.7 62.23 0)
 			(effects
@@
 			(project "Cubesat-FC-V1"
 				(path "/f01d9098-91c1-4e97-a02a-fecce6a76317/353c0638-7d15-4c84-b70a-670532d5bdf1"
-					(reference "#PWR066")
+					(reference "#PWR070")
 					(unit 1)
 				)
@@
 		(dnp no)
 		(fields_autoplaced yes)
-		(property "Reference" "#PWR064"
+		(property "Reference" "#PWR071"
 			(at 93.98 96.52 0)
 			(effects
@@
 			(project ""
 				(path "/f01d9098-91c1-4e97-a02a-fecce6a76317/353c0638-7d15-4c84-b70a-670532d5bdf1"
-					(reference "#PWR064")
+					(reference "#PWR071")
 					(unit 1)
 				)
@@
 		(on_board yes)
 		(dnp no)
-		(property "Reference" "#PWR065"
+		(property "Reference" "#PWR069"
 			(at 139.7 49.53 0)
 			(effects
@@
 			(project "Cubesat-FC-V1"
 				(path "/f01d9098-91c1-4e97-a02a-fecce6a76317/353c0638-7d15-4c84-b70a-670532d5bdf1"
-					(reference "#PWR065")
+					(reference "#PWR069")
 					(unit 1)
 				)

Commit message: more routing
Parts:
- C49, C50: voltage (none) -> 10
Changed lines of the file:
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@@
+			)
+		)
+		(property "voltage" "10"
+			(at 139.7 50.8 0)
+			(effects
+				(font
+					(size 1.27 1.27)
+				)
+				(hide yes)
 			)
 		)
@@
 			(at 148.59 50.8 0)
 			(effects
+				(font
+					(size 1.27 1.27)
+				)
+				(hide yes)
+			)
+		)
+		(property "voltage" "10"
+			(at 148.59 50.8 0)
+			(effects

Commit message: Formatting
Other:
- company: (none) -> UMASS Cubesat Lab
Changed lines of the file:
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@@
 	(generator_version "9.0")
 	(paper "A5")
+	(title_block
+		(date "2026-03-22")
+		(rev "R1")
+		(company "UMASS Cubesat Lab")
+	)
 	(junction
 		(at 139.7 54.61)
