File: CAN.kicad_sch (KiCad schematic)
At the start: 4 parts, among them U14 MCP2558FD

Commit message: Beginnings of routing
Parts:
- renumbered C71 to C70, C70 to C71, R15 to R18, U14 to U15
Changed lines of the file:
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@@
 		(dnp no)
 		(fields_autoplaced yes)
-		(property "Reference" "#PWR0108"
+		(property "Reference" "#PWR0114"
 			(at 74.93 76.2 0)
 			(effects
@@
 			(project "Cubesat-FC-V1"
 				(path "/f01d9098-91c1-4e97-a02a-fecce6a76317/005f7898-6949-46b1-b8b2-ba9d55ad0483"
+					(reference "#PWR0120")
+					(unit 1)
+				)
+				(path "/f01d9098-91c1-4e97-a02a-fecce6a76317/e1f1d40c-4f52-40ce-a497-e48f0d16f75c"
 					(reference "#PWR0114")
-					(unit 1)
-				)
-				(path "/f01d9098-91c1-4e97-a02a-fecce6a76317/e1f1d40c-4f52-40ce-a497-e48f0d16f75c"
-					(reference "#PWR0108")
 					(unit 1)
 				)
@@
 		(dnp no)
 		(fields_autoplaced yes)
-		(property "Reference" "#PWR0111"
+		(property "Reference" "#PWR0116"
 			(at 88.9 81.28 0)
 			(effects
@@
 			(project "Cubesat-FC-V1"
 				(path "/f01d9098-91c1-4e97-a02a-fecce6a76317/005f7898-6949-46b1-b8b2-ba9d55ad0483"
-					(reference "#PWR0117")
-					(unit 1)
-				)
-				(path "/f01d9098-91c1-4e97-a02a-fecce6a76317/e1f1d40c-4f52-40ce-a497-e48f0d16f75c"
-					(reference "#PWR0111")
+					(reference "#PWR0122")
+					(unit 1)
+				)
+				(path "/f01d9098-91c1-4e97-a02a-fecce6a76317/e1f1d40c-4f52-40ce-a497-e48f0d16f75c"
+					(reference "#PWR0116")
 					(unit 1)
 				)
@@
 		(on_board yes)
 		(dnp no)
-		(property "Reference" "#PWR0110"
+		(property "Reference" "#PWR0112"
 			(at 88.9 53.34 0)
 			(effects
@@
 			(project "Cubesat-FC-V1"
 				(path "/f01d9098-91c1-4e97-a02a-fecce6a76317/005f7898-6949-46b1-b8b2-ba9d55ad0483"
-					(reference "#PWR0116")
-					(unit 1)
-				)
-				(path "/f01d9098-91c1-4e97-a02a-fecce6a76317/e1f1d40c-4f52-40ce-a497-e48f0d16f75c"
-					(reference "#PWR0110")
+					(reference "#PWR0118")
+					(unit 1)
+				)
+				(path "/f01d9098-91c1-4e97-a02a-fecce6a76317/e1f1d40c-4f52-40ce-a497-e48f0d16f75c"
+					(reference "#PWR0112")
 					(unit 1)
 				)
@@
 		(on_board yes)
 		(dnp no)
-		(property "Reference" "R15"
+		(property "Reference" "R18"
 			(at 106.426 62.23 0)
 			(effects
@@
 			(project "Cubesat-FC-V1"
 				(path "/f01d9098-91c1-4e97-a02a-fecce6a76317/005f7898-6949-46b1-b8b2-ba9d55ad0483"
-					(reference "R16")
-					(unit 1)
-				)
-				(path "/f01d9098-91c1-4e97-a02a-fecce6a76317/e1f1d40c-4f52-40ce-a497-e48f0d16f75c"
-					(reference "R15")
+					(reference "R19")
+					(unit 1)
+				)
+				(path "/f01d9098-91c1-4e97-a02a-fecce6a76317/e1f1d40c-4f52-40ce-a497-e48f0d16f75c"
+					(reference "R18")
 					(unit 1)
 				)
@@
 		(on_board yes)
 		(dnp no)
-		(property "Reference" "C71"
+		(property "Reference" "C70"
 			(at 80.01 44.4562 0)
 			(effects
@@
 			(project "Cubesat-FC-V1"
 				(path "/f01d9098-91c1-4e97-a02a-fecce6a76317/005f7898-6949-46b1-b8b2-ba9d55ad0483"
-					(reference "C73")
-					(unit 1)
-				)
-				(path "/f01d9098-91c1-4e97-a02a-fecce6a76317/e1f1d40c-4f52-40ce-a497-e48f0d16f75c"
-					(reference "C71")
+					(reference "C72")
+					(unit 1)
+				)
+				(path "/f01d9098-91c1-4e97-a02a-fecce6a76317/e1f1d40c-4f52-40ce-a497-e48f0d16f75c"
+					(reference "C70")
 					(unit 1)
 				)
@@
 		(on_board yes)
 		(dnp no)
-		(property "Reference" "C70"
+		(property "Reference" "C71"
 			(at 59.69 67.3162 0)
 			(effects
@@
 			(project "Cubesat-FC-V1"
 				(path "/f01d9098-91c1-4e97-a02a-fecce6a76317/005f7898-6949-46b1-b8b2-ba9d55ad0483"
-					(reference "C72")
-					(unit 1)
-				)
-				(path "/f01d9098-91c1-4e97-a02a-fecce6a76317/e1f1d40c-4f52-40ce-a497-e48f0d16f75c"
-					(reference "C70")
+					(reference "C73")
+					(unit 1)
+				)
+				(path "/f01d9098-91c1-4e97-a02a-fecce6a76317/e1f1d40c-4f52-40ce-a497-e48f0d16f75c"
+					(reference "C71")
 					(unit 1)
 				)
@@
 		(dnp no)
 		(fields_autoplaced yes)
-		(property "Reference" "U14"
+		(property "Reference" "U15"
 			(at 91.0433 50.8 0)
 			(effects
@@
 			(project "Cubesat-FC-V1"
 				(path "/f01d9098-91c1-4e97-a02a-fecce6a76317/005f7898-6949-46b1-b8b2-ba9d55ad0483"
+					(reference "U16")
+					(unit 1)
+				)
+				(path "/f01d9098-91c1-4e97-a02a-fecce6a76317/e1f1d40c-4f52-40ce-a497-e48f0d16f75c"
 					(reference "U15")
-					(unit 1)
-				)
-				(path "/f01d9098-91c1-4e97-a02a-fecce6a76317/e1f1d40c-4f52-40ce-a497-e48f0d16f75c"
-					(reference "U14")
 					(unit 1)
 				)
@@
 		(dnp no)
 		(fields_autoplaced yes)
-		(property "Reference" "#PWR0109"
+		(property "Reference" "#PWR0111"
 			(at 82.55 55.88 0)
 			(effects
@@
 			(project "Cubesat-FC-V1"
 				(path "/f01d9098-91c1-4e97-a02a-fecce6a76317/005f7898-6949-46b1-b8b2-ba9d55ad0483"
-					(reference "#PWR0115")
-					(unit 1)
-				)
-				(path "/f01d9098-91c1-4e97-a02a-fecce6a76317/e1f1d40c-4f52-40ce-a497-e48f0d16f75c"
-					(reference "#PWR0109")
+					(reference "#PWR0117")
+					(unit 1)
+				)
+				(path "/f01d9098-91c1-4e97-a02a-fecce6a76317/e1f1d40c-4f52-40ce-a497-e48f0d16f75c"
+					(reference "#PWR0111")
 					(unit 1)
 				)
@@
 		(dnp no)
 		(fields_autoplaced yes)
-		(property "Reference" "#PWR0106"
+		(property "Reference" "#PWR0113"
 			(at 62.23 68.58 0)
 			(effects
@@
 			(project "Cubesat-FC-V1"
 				(path "/f01d9098-91c1-4e97-a02a-fecce6a76317/005f7898-6949-46b1-b8b2-ba9d55ad0483"
-					(reference "#PWR0112")
-					(unit 1)
-				)
-				(path "/f01d9098-91c1-4e97-a02a-fecce6a76317/e1f1d40c-4f52-40ce-a497-e48f0d16f75c"
-					(reference "#PWR0106")
+					(reference "#PWR0119")
+					(unit 1)
+				)
+				(path "/f01d9098-91c1-4e97-a02a-fecce6a76317/e1f1d40c-4f52-40ce-a497-e48f0d16f75c"
+					(reference "#PWR0113")
 					(unit 1)
 				)
@@
 		(dnp no)
 		(fields_autoplaced yes)
-		(property "Reference" "#PWR0107"
+		(property "Reference" "#PWR0115"
 			(at 62.23 78.74 0)
 			(effects
@@
 			(project "Cubesat-FC-V1"
 				(path "/f01d9098-91c1-4e97-a02a-fecce6a76317/005f7898-6949-46b1-b8b2-ba9d55ad0483"
-					(reference "#PWR0113")
-					(unit 1)
-				)
-				(path "/f01d9098-91c1-4e97-a02a-fecce6a76317/e1f1d40c-4f52-40ce-a497-e48f0d16f75c"
-					(reference "#PWR0107")
-					(unit 1)
-				)
+					(reference "#PWR0121")
+					(unit 1)
+				)
+				(path "/f01d9098-91c1-4e97-a02a-fecce6a76317/e1f1d40c-4f52-40ce-a497-e48f0d16f75c"
+					(reference "#PWR0115")
+					(unit 1)
+				)

Commit message: Finish initial revision
Connections:
- net +3V3 is gone; now on net +3.3V: C71.1, U15.5 (VIO)
Changed lines of the file:
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@@
+	)
+	(symbol
+		(lib_id "power:+3.3V")
+		(at 62.23 64.77 0)
+		(unit 1)
+		(exclude_from_sim no)
+		(in_bom yes)
+		(on_board yes)
+		(dnp no)
+		(property "Reference" "#PWR034"
+			(at 62.23 68.58 0)
+			(effects
+				(font
+					(size 1.27 1.27)
+				)
+				(hide yes)
+			)
+		)
+		(property "Value" "+3.3V"
+			(at 62.23 59.69 0)
+			(effects
+				(font
+					(size 1.27 1.27)
+				)
+			)
+		)
+		(property "Footprint" ""
+			(at 62.23 64.77 0)
+			(effects
+				(font
+					(size 1.27 1.27)
+				)
+				(hide yes)
+			)
+		)
+		(property "Datasheet" ""
+			(at 62.23 64.77 0)
+			(effects
+				(font
+					(size 1.27 1.27)
+				)
+				(hide yes)
+			)
+		)
+		(property "Description" "Power symbol creates a global label with name \"+3.3V\""
+			(at 62.23 64.77 0)
+			(effects
+				(font
+					(size 1.27 1.27)
+				)
+				(hide yes)
+			)
+		)
+		(pin "1"
+		)
+		(instances
+			(project "Cubesat-FC-V1"
+				(path "/f01d9098-91c1-4e97-a02a-fecce6a76317/005f7898-6949-46b1-b8b2-ba9d55ad0483"
+					(reference "#PWR035")
+					(unit 1)
+				)
+				(path "/f01d9098-91c1-4e97-a02a-fecce6a76317/e1f1d40c-4f52-40ce-a497-e48f0d16f75c"
+					(reference "#PWR034")
+					(unit 1)
+				)
+			)
+		)
 	)
 	(symbol
@@
 					(unit 1)
 				)
-			)
-		)
-	)
-	(symbol
-		(lib_id "power:+3V3")
-		(at 62.23 64.77 0)
-		(unit 1)
-		(exclude_from_sim no)
-		(in_bom yes)
-		(on_board yes)
-		(dnp no)
-		(fields_autoplaced yes)
-		(property "Reference" "#PWR0113"
-			(at 62.23 68.58 0)
-			(effects
-				(font
-					(size 1.27 1.27)
-				)
-				(hide yes)
-			)
-		)
-		(property "Value" "+3V3"
-			(at 62.23 59.69 0)
-			(effects
-				(font
-					(size 1.27 1.27)
-				)
-			)
-		)
-		(property "Footprint" ""
-			(at 62.23 64.77 0)
-			(effects
-				(font
-					(size 1.27 1.27)
-				)
-				(hide yes)
-			)
-		)
-		(property "Datasheet" ""
-			(at 62.23 64.77 0)
-			(effects
-				(font
-					(size 1.27 1.27)
-				)
-				(hide yes)
-			)
-		)
-		(property "Description" "Power symbol creates a global label with name \"+3V3\""
-			(at 62.23 64.77 0)
-			(effects
-				(font
-					(size 1.27 1.27)
-				)
-				(hide yes)
-			)
-		)
-		(pin "1"
-		)
-		(instances
-			(project "Cubesat-FC-V1"
-				(path "/f01d9098-91c1-4e97-a02a-fecce6a76317/005f7898-6949-46b1-b8b2-ba9d55ad0483"
-					(reference "#PWR0119")
-					(unit 1)
-				)
-				(path "/f01d9098-91c1-4e97-a02a-fecce6a76317/e1f1d40c-4f52-40ce-a497-e48f0d16f75c"
-					(reference "#PWR0113")
-					(unit 1)
-				)

Commit message: Formatting
Other:
- company: (none) -> UMASS Cubesat Lab
Changed lines of the file:
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@@
 	(generator_version "9.0")
 	(paper "A5")
+	(title_block
+		(date "2026-03-22")
+		(rev "R1")
+		(company "UMASS Cubesat Lab")
+	)
 	(junction
 		(at 88.9 50.8)

Commit message: R1 candidate
Parts:
- removed C71: 10u, Capacitor_SMD:C_0402_1005Metric, symbol Device:C_Small
- removed U15: MCP2558FD, Package_SO:SOIC-8_3.9x4.9mm_P1.27mm, symbol Interface_CAN_LIN:MCP2558FD-xSN
- added U15: TCAN330, Package_TO_SOT_SMD:SOT-23-8, symbol Interface_CAN_LIN:TCAN330
Connections:
- net +3.3V: now also U15.3 (VCC)
- net CAN_H: now also U15.7 (CANH)
- net CAN_L: now also U15.6 (CANL)
- net GND: now also U15.2 (GND), U15.5 (SHDN), U15.8 (S)
- net RX_CAN: now also U15.4 (RXD)
- net TX_CAN: now also U15.1 (TXD)
Other:
- moved on the sheet: C70
