File: Cubesat-FC-V1.kicad_pcb (KiCad board)
At the start: 4 copper layers, 75 x 75 mm, 223 parts, among them J1 Conn_01x03_Pin, J10 Conn_01x04_Pin, J11 USB_C_Receptacle_USB2.0_14P, J12 Conn_01x03_Pin, J13 Conn_01x03_Pin, J16 Screw_Terminal_01x02, J2 Conn_ST_STDC14, J3 Conn_01x03_Pin, J4 Conn_01x04_Pin, J5 Conn_01x04_Pin, J6 Conn_01x04_Pin, J7 USB_C_Receptacle_USB2.0_14P, J8 Conn_01x04_Pin, J9 Micro_SD_Card, SW1 SW_SPDT, SW2 SW_SPDT, SW3 SW_DIP_x04, SW4 SW_Button, SW5 SW_SPDT, SW6 SW_SPDT, U11 W25Q128JVS, U12 W25Q128JVS, U13 W25Q128JVS, U14 W25Q128JVS, U15 MCP2558FD, U16 MCP2558FD, U18 CP2102N-Axx-xQFN24, U2 TPS2117DRL, U3 TPS62933, U4 STM32H757BITx, U6 W25Q128JVS, U8 MMC5983MA, Y1 32.768KHZ, Y2 ASCO, Y3 ASE-xxxMHz

Commit message: R1 candidate
Parts:
- removed C71, C73: 10u, Capacitor_SMD:C_0402_1005Metric
- added R26: 20k, Resistor_SMD:R_0402_1005Metric, B.Cu at (151.2, 81.4)
- added R27: 47k, Resistor_SMD:R_0402_1005Metric, B.Cu at (151.2, 82.4)
- C47, C48: value ?? -> 15p
- FB1: value ??? -> 600ohm@1mhz
- J1, J12, J13, J3: value Conn_01x03_Pin -> 53253-0370
- J10, J4, J5, J6, J8: value Conn_01x04_Pin -> 53253-0470
- R1, R2, R3, R4, R5, R6: value R_Small -> 1k
- R11: value R_Small -> 10k
- U15, U16: value MCP2558FD -> TCAN330; footprint Package_SO:SOIC-8_3.9x4.9mm_P1.27mm -> Package_TO_SOT_SMD:SOT-23-8
- Y2: value ASCO -> 24MHZ
- moved C43 25.1 mm to (157.6, 78.7), turned to 0 degrees
- moved C44 25.1 mm to (133.2, 72.9), turned to 90 degrees
- moved U15 1.60 mm to (139.0, 65.4)
- moved U16 1.60 mm to (132.8, 65.4)
Connections:
- net +5V renamed /3V3_EXT
- net /STM32H747/FMCNBL0 renamed /SDRAM/FMCLQDM
- net /STM32H747/FMCNBL1 renamed /SDRAM/FMCUQDM
- C2 pad 1: /BUCKVIN -> VBUS
- C3 pad 1: /BUCKVIN -> VBUS
- C4 pad 1: /BUCKVIN -> VBUS
- C42 pad 1: /STM32H747/VCAP -> /STM32H747/VCAP0
- C43 pad 1: /STM32H747/VCAP -> /STM32H747/VCAP1
- C44 pad 1: /STM32H747/VCAP -> /STM32H747/VCAP2
- J11 pad S1: unconnected-(J11-SHIELD-PadS1)_3 -> GND
- J7 pad S1: unconnected-(J7-SHIELD-PadS1)_2 -> GND
- L1 pad 2: +3.3V -> /BUCKVOUT
- R13 pad 1: +3.3V -> /BUCKVOUT
- U11 pad 3: unconnected-(U11-IO2-Pad3) -> +3.3V
- U11 pad 7: unconnected-(U11-IO3-Pad7) -> +3.3V
- U12 pad 3: unconnected-(U12-IO2-Pad3) -> +3.3V
- U12 pad 7: unconnected-(U12-IO3-Pad7) -> +3.3V
- U13 pad 3: unconnected-(U13-IO2-Pad3) -> +3.3V
- U13 pad 7: unconnected-(U13-IO3-Pad7) -> +3.3V
- U14 pad 3: unconnected-(U14-IO2-Pad3) -> +3.3V
- U14 pad 7: unconnected-(U14-IO3-Pad7) -> +3.3V
- U15 pad 5: +3.3V -> GND
- U16 pad 5: +3.3V -> GND
- U2 pad 2: /BUCKVIN -> +3.3V
- U2 pad 6: VBUS -> /BUCKVOUT
- U2 pad 7: /BUCKVIN -> +3.3V
- U3 pad 3: /BUCKVIN -> VBUS
- U4 pad 147: /STM32H747/USB_FS_VBUS -> /USB_FS_VBUS
- U4 pad 152: /STM32H747/VCAP -> /STM32H747/VCAP1
- U4 pad 199: /STM32H747/VCAP -> /STM32H747/VCAP2
- U4 pad 89: /STM32H747/VCAP -> /STM32H747/VCAP0
Routing:
- net VBUS: track 60.9 -> 107.4 mm, vias 0 -> 2
- net +3.3V: track 92.1 -> 129.2 mm
- net /BUCKVOUT: track 0.00 -> 29.4 mm, vias 0 -> 6
- net /STM32H747/VCAP: track 4.56 -> 0.00 mm
- net /BUCKVIN: track 11.6 -> 7.86 mm
- net /CAN Transceiver/TX_CAN: track 5.66 -> 9.02 mm
- net /CAN Transceiver1/RX_CAN: track 5.37 -> 8.69 mm
- net GND: track 135.3 -> 133.0 mm, vias 725 -> 92
- net /STM32H747/VCAP2: track 0.00 -> 1.63 mm
- net /SWD_TRACE_D3: track 40.5 -> 38.9 mm
- net /CAN Transceiver1/TX_CAN: track 7.81 -> 9.29 mm
- net /PIN_PROC1GP1: track 18.9 -> 20.4 mm, vias 3 -> 2
- net /STM32H747/VCAP0: track 0.00 -> 1.47 mm
- net /STM32H747/VCAP1: track 0.00 -> 1.47 mm
- net /SDRAM/FMCCAS: track 40.1 -> 38.6 mm, vias 3 -> 2
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- added copper zone on F.Cu, net VBUS
- removed copper zone on F.Cu, net /BUCKVIN
