File: Cubesat-FC-V1.kicad_sch (KiCad schematic)
At the start: 64 parts, among them J1 Conn_01x04_Pin, J2 Conn_01x04_Pin, J3 Conn_01x04_Pin, J4 Conn_01x03_Pin, J5 Conn_01x04_Pin, J6 Conn_ST_STDC14, J7 Conn_01x03_Pin, J8 USB_C_Receptacle_USB2.0_14P, SW1 SW_DIP_x04, SW2 SW_SPDT, SW3 SW_SPDT, SW4 SW_SPDT, SW5 SW_Button, SW6 SW_SPDT, U2 TPS62933

Commit message: Beginnings of routing
Parts:
- removed JP1, JP3: Jumper_3_Open, Jumper:SolderJumper-3_P1.3mm_Open_RoundedPad1.0x1.5mm, symbol Jumper:Jumper_3_Open
- added C74, C77: 10u, Capacitor_SMD:C_0402_1005Metric, symbol Device:C_Small
- added C75, C76: 0.1u, Capacitor_SMD:C_0402_1005Metric, symbol Device:C_Small
- added D7: LED_G, LED_SMD:LED_0603_1608Metric, symbol Device:D_Small
- added D8: LED_R, LED_SMD:LED_0603_1608Metric, symbol Device:D_Small
- added H1, H2, H3, H4: M3, MountingHole:MountingHole_3.2mm_M3_ISO7380_Pad_TopBottom, symbol Mechanical:MountingHole_Pad
- added J10: Conn_01x04_Pin, Connector_Molex:Molex_Micro-Latch_53253-0470_1x04_P2.00mm_Vertical, symbol Connector:Conn_01x04_Pin
- added J11: USB_C_Receptacle_USB2.0_14P, Connector_USB:USB_C_Receptacle_GCT_USB4105-xx-A_16P_TopMnt_Horizontal, symbol Connector:USB_C_Receptacle_USB2.0_14P
- added J12, J13, J14, J15: Conn_01x03_Pin, Connector_Molex:Molex_Micro-Latch_53253-0370_1x03_P2.00mm_Vertical, symbol Connector:Conn_01x03_Pin
- added R10, R9: 1k, Resistor_SMD:R_0402_1005Metric, symbol Device:R_Small
- added R11: R_Small, Resistor_SMD:R_0402_1005Metric, symbol Device:R_Small
- added R20, R22, R23: 20k, Resistor_SMD:R_0402_1005Metric, symbol Device:R_Small
- added R21: 47k, Resistor_SMD:R_0402_1005Metric, symbol Device:R_Small
- added R24, R25: 5.1k, Resistor_SMD:R_0402_1005Metric, symbol Device:R_Small
- added TP10, TP11, TP12, TP13, TP14, TP15, TP16, TP17, TP18, TP19, TP20, TP21, TP22, TP23, TP24, TP7, TP8, TP9: TestPoint, TestPoint:TestPoint_Pad_D1.5mm, symbol Connector:TestPoint
- added U18: CP2102N-Axx-xQFN24, Package_DFN_QFN:QFN-24-1EP_4x4mm_P0.5mm_EP2.6x2.6mm, symbol Interface_USB:CP2102N-Axx-xQFN24
- added U2: TPS2117DRL, Package_TO_SOT_SMD:SOT-583-8, symbol Power_Management:TPS2116DRL
- BZ1: footprint (none) -> Buzzer_Beeper:Buzzer_Murata_PKMCS0909E
- J1: renamed from J7; footprint (none) -> Connector_Molex:Molex_Micro-Latch_53253-0370_1x03_P2.00mm_Vertical
- J3: renamed from J4; footprint (none) -> Connector_Molex:Molex_Micro-Latch_53253-0370_1x03_P2.00mm_Vertical
- J4: renamed from J1; footprint (none) -> Connector_Molex:Molex_Micro-Latch_53253-0470_1x04_P2.00mm_Vertical
- J5: footprint (none) -> Connector_Molex:Molex_Micro-Latch_53253-0470_1x04_P2.00mm_Vertical
- J6: renamed from J3; footprint (none) -> Connector_Molex:Molex_Micro-Latch_53253-0470_1x04_P2.00mm_Vertical
- J7: renamed from J8; footprint (none) -> Connector_USB:USB_C_Receptacle_GCT_USB4105-xx-A_16P_TopMnt_Horizontal
- J8: renamed from J2; footprint (none) -> Connector_Molex:Molex_Micro-Latch_53253-0470_1x04_P2.00mm_Vertical
- JP2: renamed from JP7; footprint (none) -> Jumper:SolderJumper-3_P1.3mm_Open_RoundedPad1.0x1.5mm
- JP3: renamed from JP9; footprint (none) -> Jumper:SolderJumper-3_P1.3mm_Open_RoundedPad1.0x1.5mm
- JP5: renamed from JP8; footprint (none) -> Jumper:SolderJumper-3_P1.3mm_Open_RoundedPad1.0x1.5mm
- R12: renamed from R1; footprint (none) -> Resistor_SMD:R_0402_1005Metric
- SW1: renamed from SW2; footprint Button_Switch_SMD:SW_DPDT_CK_JS202011JCQN -> Button_Switch_THT:SW_CK_JS202011CQN_DPDT_Straight
- SW2: renamed from SW6; footprint Button_Switch_SMD:SW_DPDT_CK_JS202011JCQN -> Button_Switch_THT:SW_CK_JS202011CQN_DPDT_Straight
- SW5: renamed from SW3; footprint Button_Switch_SMD:SW_DPDT_CK_JS202011JCQN -> Button_Switch_THT:SW_CK_JS202011CQN_DPDT_Straight
- SW6: renamed from SW4; footprint Button_Switch_SMD:SW_DPDT_CK_JS202011JCQN -> Button_Switch_THT:SW_CK_JS202011CQN_DPDT_Straight
- TP1, TP2, TP3, TP4, TP5, TP6: footprint TestPoint:TestPoint_Pad_1.5x1.5mm -> TestPoint:TestPoint_Pad_D1.5mm
- U1: footprint (none) -> Connector_PinSocket_2.54mm:PinSocket_2x10_P2.54mm_Vertical
- renumbered C5 to C1, C1 to C2, C2 to C3, C3 to C4, C4 to C5, J6 to J2, JP4 to JP6, JP6 to JP7, JP2 to JP8, JP5 to JP9, R5 to R1, R4 to R15, R2 to R16, R3 to R17, R6 to R2, R7 to R3, R8 to R4, R9 to R5, R10 to R6, R11 to R7, R12 to R8, SW1 to SW3, SW5 to SW4, U2 to U3
Connections:
- net +3.3V: now also J10.1 (Pin_1)
- net BUCKVIN: now also U2.2 (VOUT), U2.7 (VOUT)
- net BUZZER: now also BZ1.1 (+), SW1.1 (A); no longer R12.1
- net CAN1_H: now also J13.1 (Pin_1), J15.1 (Pin_1)
- net CAN1_L: now also J13.3 (Pin_3), J15.3 (Pin_3)
- net CAN2_H: now also J12.1 (Pin_1), J14.1 (Pin_1)
- net CAN2_L: now also J12.3 (Pin_3), J14.3 (Pin_3)
- net GND: now also C74.2, C75.2, C76.2, C77.2, H1.1, H2.1, H3.1, H4.1, J10.4 (Pin_4), J11.A1 (GND), J11.A12 (GND), J11.B1 (GND), J11.B12 (GND), J12.2 (Pin_2), J13.2 (Pin_2), J14.2 (Pin_2), J15.2 (Pin_2), R10.2, R21.1, R24.2, R25.1, U18.2 (GND), U18.25 (GND), U2.1 (GND)
- net I2C2_SDA: now also TP24.1; no longer J8.3 (Pin_3)
- net UART4_RX: now also U18.20 (RXD)
- net UART4_TX: now also U18.21 (TXD)
- net VBUS: now also C74.1, C75.1, J11.A4 (VBUS), J11.A9 (VBUS), J11.B4 (VBUS), J11.B9 (VBUS), R20.1, U18.7 (VREGIN), U2.6 (VIN2)
- net BUCK_EN: now reaches JP2.2 (C), U3.2 (EN)
- net at JP9.1 (A): now also JP7.2 (C)
- net ISC2_SCL renamed I2C2_SCL
- net I2C2_SCL: now also TP23.1; no longer J8.2 (Pin_2)
- net STM32H747/PIN_CONFIG_0 renamed PIN_GPIO_CFG_0
- net STM32H747/PIN_CONFIG_1 renamed PIN_GPIO_CFG_1
- net STM32H747/PIN_CONFIG_2 renamed PIN_GPIO_CFG_2
- net STM32H747/PIN_CONFIG_3 renamed PIN_GPIO_CFG_3
- new net: R20.2, R21.2, U18.8 (VBUS)
- new net: R10.1, R9.1, U2.4 (PR1)
- new net: D8.1 (K), U18.13 (~{RXT}/GPIO.1)
- new net: D8.2 (A), R23.1
- new net: R11.1, U2.8 (ST)
- new net: J11.A5 (CC1), R25.2
- new net: J11.B5 (CC2), R24.1
- new net: D7.1 (K), U18.14 (~{TXT}/GPIO.0)
- new net: D7.2 (A), R22.1
- new net +5V: R11.2, R9.2, U2.3 (VIN1), U2.5 (MODE)
- new net 3.3V_BRIDGE: C76.1, C77.1, R22.2, R23.2, U18.5 (VIO), U18.6 (VDD)
- new net BRIDGE_DM: J11.A7 (D-), J11.B7 (D-), U18.4 (D-)
- new net BRIDGE_DP: J11.A6 (D+), J11.B6 (D+), U18.3 (D+)
- new net BRIDGE_NRST: U18.9 (~{RST})
- new net I2C3_SCL: J10.2 (Pin_2), J8.2 (Pin_2), TP21.1
- new net I2C3_SDA: J10.3 (Pin_3), J8.3 (Pin_3), TP22.1
- new net PIN_GPIO_BUZZER: R12.1
- new net SPI1_CIPO: TP16.1
- new net SPI1_COPI: TP15.1
- new net SPI1_SCK: TP14.1
- new net SPI2_CIPO: TP12.1
- new net SPI2_COPI: TP11.1
- new net SPI2_SCK: TP13.1
- new net SPI_CS_CATALOG0: TP17.1
- new net SPI_CS_CATALOG1: TP18.1
- new net SPI_CS_CATALOG2: TP19.1
- new net SPI_CS_DATALOG: TP20.1
- new net SPI_CS_IMU_PRI: TP10.1
- new net SPI_CS_IMU_SEC0: TP9.1
- new net SPI_CS_IMU_SEC1: TP8.1
- new net SPI_CS_MAG: TP7.1
- no-connect marks 3 -> 14
Other:
- sheet Flash Storage ports: added SPI_CS_DATALOG; removed SPI_CS_DATALOG0
- sheet SDRAM ports: added FMCA[0..12], FMCD[0..15]; removed FMC{A[0..12] D[0..15]}
- sheet STM32H747 ports: added FDCAN1_RX, FDCAN1_TX, FMCA[0..12], FMCD[0..15], I2C3_SCL, I2C3_SDA, UART4_RX, UART4_TX, USB_FS_VBUS; removed FDCAN1_RX/UART4_RX, FDCAN1_TX/UART4_TX, FMC{A[0..12] D[0..15]}
- note added: "3.3v buck converter"
- note added: "Do these need to be swapped?"
- note added: "I/O connection"
- note added: "Power configuration"
- note added: "Power source selection"
- note added: "STM32 I/O configuration"
- note added: "STM32 low level configuration"
- note added: "State indication"
- note removed: "Configuration"
- note removed: "Swappable between CAN / Debug UART"
- moved on the sheet: BZ1, C1, C10, C11, C2, C3, C4, C5, C6, C7, C8, C9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

Commit message: more routing
Parts:
- removed C11: 100u, Capacitor_SMD:C_1206_3216Metric, symbol Device:C_Small
- removed J14, J15: Conn_01x03_Pin, Connector_Molex:Molex_Micro-Latch_53253-0370_1x03_P2.00mm_Vertical, symbol Connector:Conn_01x03_Pin
- removed JP3, JP5: Jumper_3_Open, Jumper:SolderJumper-3_P1.3mm_Open_RoundedPad1.0x1.5mm, symbol Jumper:Jumper_3_Open
- removed JP6, JP7, JP8, JP9: Jumper, Jumper:SolderJumper-3_P1.3mm_Open_RoundedPad1.0x1.5mm, symbol Jumper:Jumper_3_Open
- added J16: Screw_Terminal_01x02, TerminalBlock_Phoenix:TerminalBlock_Phoenix_MKDS-1,5-2-5.08_1x02_P5.08mm_Horizontal, symbol Connector:Screw_Terminal_01x02
- C1, C5, C74, C75, C76, C77: voltage (none) -> 10
- C10, C2, C8, C9: voltage (none) -> 30
- C3, C4, C6, C7: footprint Capacitor_SMD:C_0402_1005Metric -> Capacitor_SMD:C_1206_3216Metric; voltage (none) -> 30
- L1: value 7.8u -> 5.6u; footprint (none) -> Inductor_SMD:L_Coilcraft_XAL7070-XXX
- R1, R10, R11, R12, R13, R14, R15, R16, R17, R2, R20, R21, R22, R23, R24, R25, R3, R4, R5, R6, R7, R8, R9: voltage (none) -> 50
Connections:
- net +3.3V: now also C10.1, C6.1, C7.1, C8.1, C9.1
- net +5V: now also J16.1 (Pin_1)
- net BUCKVIN: now also JP2.3 (B)
- net GND: now also J16.2 (Pin_2)
- net at SW5.2 (B): now also R16.2
- net at R17.2: now also SW6.2 (B)
- net at JP2.1 (A): now also SW2.2 (B)
- removed net 3V3_BUCK: C1.2, C10.1, C6.1, C7.1, C8.1, C9.1, L1.1, U3.5 (SW)
- new net: C1.2, L1.1, U3.5 (SW)
Other:
- moved on the sheet: SW2, SW5, SW6

Commit message: more routing
Connections:
- net +3.3V: now also L1.2, R13.1
Changed lines of the file:
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@@
 	)
 	(junction
-		(at 330.2 196.85)
+		(at 393.7 204.47)
 		(diameter 0)
 		(color 0 0 0 0)
 	)
 	(junction
-		(at 386.08 196.85)
+		(at 330.2 196.85)
 		(diameter 0)
 		(color 0 0 0 0)
@@
 	(wire
 		(pts
-			(xy 387.35 195.58) (xy 387.35 196.85)
+			(xy 394.97 203.2) (xy 394.97 204.47)
 		)
 		(stroke
@@
 	(wire
 		(pts
-			(xy 386.08 196.85) (xy 387.35 196.85)
+			(xy 393.7 204.47) (xy 394.97 204.47)
 		)
 		(stroke
@@
 					(unit 1)
 				)
+			)
+		)
+	)
+	(symbol
+		(lib_id "power:+3.3V")
+		(at 394.97 203.2 0)
+		(mirror y)
+		(unit 1)
+		(exclude_from_sim no)
+		(in_bom yes)
+		(on_board yes)
+		(dnp no)
+		(fields_autoplaced yes)
+		(property "Reference" "#PWR027"
+			(at 394.97 207.01 0)
+			(effects
+				(font
+					(size 1.27 1.27)
+				)
+				(hide yes)
+			)
+		)
+		(property "Value" "+3.3V"
+			(at 394.97 198.12 0)
+			(effects
+				(font
+					(size 1.27 1.27)
+				)
+			)
+		)
+		(property "Footprint" ""
+			(at 394.97 203.2 0)
+			(effects
+				(font
+					(size 1.27 1.27)
+				)
+				(hide yes)
+			)
+		)
+		(property "Datasheet" ""
+			(at 394.97 203.2 0)
+			(effects
+				(font
+					(size 1.27 1.27)
+				)
+				(hide yes)
+			)
+		)
+		(property "Description" "Power symbol creates a global label with name \"+3.3V\""
+			(at 394.97 203.2 0)
+			(effects
+				(font
+					(size 1.27 1.27)
+				)
+				(hide yes)
+			)
+		)
+		(pin "1"
+		)
+		(instances
+			(project "Cubesat-FC-V1"
+				(path "/f01d9098-91c1-4e97-a02a-fecce6a76317"
+					(reference "#PWR027")
+					(unit 1)
+				)

Commit message: Finish initial revision
Parts:
- J2: footprint (none) -> Connector_PinHeader_2.54mm:PinHeader_2x07_P2.54mm_Vertical
- U1: footprint Connector_PinSocket_2.54mm:PinSocket_2x10_P2.54mm_Vertical -> Connector_PinHeader_2.54mm:PinHeader_2x10_P2.54mm_Vertical
Changed lines of the file:
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@@
 			)
 		)
-		(property "Description" "Generic connector, single row, 01x04, script generated"
+		(property "Description" "53253-0470"
 			(at 386.08 90.17 0)
 			(effects
@@
 			)
 		)
-		(property "Description" "Generic connector, single row, 01x04, script generated"
+		(property "Description" "53253-0470"
 			(at 354.33 166.37 0)
 			(effects
@@
 			)
 		)
-		(property "Description" "Generic connector, single row, 01x04, script generated"
+		(property "Description" "53253-0470"
 			(at 386.08 158.75 0)
 			(effects
@@
 			)
 		)
-		(property "Description" "Generic connector, single row, 01x03, script generated"
+		(property "Description" "53253-0370"
 			(at 424.18 53.34 0)
 			(effects
@@
 			)
 		)
-		(property "Description" "Generic connector, single row, 01x04, script generated"
+		(property "Description" "53253-0470"
 			(at 386.08 135.89 0)
 			(effects
@@
 			)
 		)
-		(property "Description" "Generic connector, single row, 01x03, script generated"
+		(property "Description" "53253-0370"
 			(at 386.08 69.85 0)
 			(effects
@@
 			)
 		)
-		(property "Description" "Generic connector, single row, 01x03, script generated"
+		(property "Description" "53253-0370"
 			(at 424.18 69.85 0)
 			(effects
@@
 			)
 		)
-		(property "Footprint" ""
+		(property "Footprint" "Connector_PinHeader_2.54mm:PinHeader_2x07_P2.54mm_Vertical"
 			(at 341.63 59.69 0)
 			(effects
@@
 			)
 		)
-		(property "Description" "Generic connector, single row, 01x04, script generated"
+		(property "Description" "53253-0470"
 			(at 386.08 113.03 0)
 			(effects
@@
 			)
 		)
-		(property "Description" "Generic connector, single row, 01x03, script generated"
+		(property "Description" "53253-0370"
 			(at 386.08 53.34 0)
 			(effects
@@
 			)
 		)
-		(property "Footprint" "Connector_PinSocket_2.54mm:PinSocket_2x10_P2.54mm_Vertical"
+		(property "Footprint" "Connector_PinHeader_2.54mm:PinHeader_2x10_P2.54mm_Vertical"
 			(at 341.63 100.33 0)
 			(effects

Commit message: Formatting
Parts:
- J1, J12, J13, J3: value Conn_01x03_Pin -> 53253-0370
- J10, J4, J5, J6, J8: value Conn_01x04_Pin -> 53253-0470
Other:
- note added: "TODO: add usb detection for STM32"
- note added: "Test Points"
- note added: "USB UART Bridge"
- company: (none) -> UMASS Cubesat Lab
- title: (none) -> UMASS Cubesat Flight Computer
- moved on the sheet: BZ1, C74, C75, C76, C77, D1, D2, D3, D4, D5, D6, D7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

Commit message: R1 candidate
Parts:
- added R26: 20k, Resistor_SMD:R_0402_1005Metric, symbol Device:R_Small
- added R27: 47k, Resistor_SMD:R_0402_1005Metric, symbol Device:R_Small
- R1, R2, R3, R4, R5, R6: value R_Small -> 1k
- R11: value R_Small -> 10k
Connections:
- net +3.3V: now also U2.2 (VOUT), U2.7 (VOUT); no longer L1.2, R13.1
- net BUCKVIN: no longer C2.1, C3.1, C4.1, U2.2 (VOUT), U2.7 (VOUT), U3.3 (VIN)
- net GND: now also J11.S1 (SHIELD), J7.S1 (SHIELD), R27.1
- net VBUS: now also C2.1, C3.1, C4.1, U3.3 (VIN), R26.1; no longer U2.6 (VIN2)
- net +5V renamed 3V3_EXT
- new net BUCKVOUT: L1.2, R13.1, U2.6 (VIN2)
- new net USB_FS_VBUS: R26.2, R27.2
- no-connect marks 14 -> 12
Other:
- moved on the sheet: C10, C6, C7, C8, C9, R10, R11, R9, U2
