File: Flash.kicad_sch (KiCad schematic)
At the start: 8 parts, among them U10 W25Q128JVS, U11 W25Q128JVS, U12 W25Q128JVS, U13 W25Q128JVS

Commit message: Beginnings of routing
Parts:
- renumbered U10 to U13, U13 to U14
Connections:
- net SPI_CS_CATALOG3 renamed SPI_CS_DATALOG
- net SPI_CS_DATALOG0 renamed SPI_CS_CATALOG0
Changed lines of the file:
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@@
 		)
 	)
-	(hierarchical_label "SPI_CS_CATALOG3"
+	(hierarchical_label "SPI_CS_DATALOG"
 		(shape input)
 		(at 101.6 35.56 180)
@@
 		)
 	)
-	(hierarchical_label "SPI_CS_DATALOG0"
+	(hierarchical_label "SPI_CS_CATALOG0"
 		(shape input)
 		(at 39.37 35.56 180)
@@
 		(dnp no)
 		(fields_autoplaced yes)
-		(property "Reference" "#PWR098"
+		(property "Reference" "#PWR0107"
 			(at 63.5 124.46 0)
 			(effects
@@
 			(project "Cubesat-FC-V1"
 				(path "/f01d9098-91c1-4e97-a02a-fecce6a76317/f101efa4-b1f1-437b-925a-4b89d5595dc0"
-					(reference "#PWR098")
+					(reference "#PWR0107")
 					(unit 1)
 				)
@@
 		(dnp no)
 		(fields_autoplaced yes)
-		(property "Reference" "#PWR096"
+		(property "Reference" "#PWR0100"
 			(at 53.34 55.88 0)
 			(effects
@@
 			(project "Cubesat-FC-V1"
 				(path "/f01d9098-91c1-4e97-a02a-fecce6a76317/f101efa4-b1f1-437b-925a-4b89d5595dc0"
-					(reference "#PWR096")
+					(reference "#PWR0100")
 					(unit 1)
 				)
@@
 		(on_board yes)
 		(dnp no)
-		(property "Reference" "U10"
+		(property "Reference" "U13"
 			(at 43.18 68.58 0)
 			(effects
@@
 			(project "Cubesat-FC-V1"
 				(path "/f01d9098-91c1-4e97-a02a-fecce6a76317/f101efa4-b1f1-437b-925a-4b89d5595dc0"
-					(reference "U10")
+					(reference "U13")
 					(unit 1)
 				)
@@
 		(dnp no)
 		(fields_autoplaced yes)
-		(property "Reference" "#PWR0101"
+		(property "Reference" "#PWR0103"
 			(at 115.57 71.12 0)
 			(effects
@@
 			(project "Cubesat-FC-V1"
 				(path "/f01d9098-91c1-4e97-a02a-fecce6a76317/f101efa4-b1f1-437b-925a-4b89d5595dc0"
-					(reference "#PWR0101")
+					(reference "#PWR0103")
 					(unit 1)
 				)
@@
 		(dnp no)
 		(fields_autoplaced yes)
-		(property "Reference" "#PWR095"
+		(property "Reference" "#PWR098"
 			(at 53.34 30.48 0)
 			(effects
@@
 			(project "Cubesat-FC-V1"
 				(path "/f01d9098-91c1-4e97-a02a-fecce6a76317/f101efa4-b1f1-437b-925a-4b89d5595dc0"
-					(reference "#PWR095")
+					(reference "#PWR098")
 					(unit 1)
 				)
@@
 		(dnp no)
 		(fields_autoplaced yes)
-		(property "Reference" "#PWR094"
+		(property "Reference" "#PWR0104"
 			(at 52.07 96.52 0)
 			(effects
@@
 			(project "Cubesat-FC-V1"
 				(path "/f01d9098-91c1-4e97-a02a-fecce6a76317/f101efa4-b1f1-437b-925a-4b89d5595dc0"
-					(reference "#PWR094")
+					(reference "#PWR0104")
 					(unit 1)
 				)
@@
 		(dnp no)
 		(fields_autoplaced yes)
-		(property "Reference" "#PWR093"
+		(property "Reference" "#PWR0102"
 			(at 52.07 71.12 0)
 			(effects
@@
 			(project "Cubesat-FC-V1"
 				(path "/f01d9098-91c1-4e97-a02a-fecce6a76317/f101efa4-b1f1-437b-925a-4b89d5595dc0"
-					(reference "#PWR093")
+					(reference "#PWR0102")
 					(unit 1)
 				)
@@
 		(on_board yes)
 		(dnp no)
-		(property "Reference" "U13"
+		(property "Reference" "U14"
 			(at 106.68 68.58 0)
 			(effects
@@
 			(project "Cubesat-FC-V1"
 				(path "/f01d9098-91c1-4e97-a02a-fecce6a76317/f101efa4-b1f1-437b-925a-4b89d5595dc0"
-					(reference "U13")
+					(reference "U14")
 					(unit 1)
 				)
@@
 		(dnp no)
 		(fields_autoplaced yes)
-		(property "Reference" "#PWR0100"
+		(property "Reference" "#PWR0101"
 			(at 115.57 55.88 0)
 			(effects
@@
 			(project "Cubesat-FC-V1"
 				(path "/f01d9098-91c1-4e97-a02a-fecce6a76317/f101efa4-b1f1-437b-925a-4b89d5595dc0"
-					(reference "#PWR0100")
+					(reference "#PWR0101")
 					(unit 1)
 				)
@@
 		(dnp no)
 		(fields_autoplaced yes)
-		(property "Reference" "#PWR0102"
+		(property "Reference" "#PWR0105"
 			(at 115.57 96.52 0)
 			(effects
@@
 			(project "Cubesat-FC-V1"
 				(path "/f01d9098-91c1-4e97-a02a-fecce6a76317/f101efa4-b1f1-437b-925a-4b89d5595dc0"
-					(reference "#PWR0102")
+					(reference "#PWR0105")
 					(unit 1)
 				)
@@
 		(dnp no)
 		(fields_autoplaced yes)
-		(property "Reference" "#PWR097"
+		(property "Reference" "#PWR0106"
 			(at 63.5 111.76 0)
 			(effects
@@
 			(project "Cubesat-FC-V1"
 				(path "/f01d9098-91c1-4e97-a02a-fecce6a76317/f101efa4-b1f1-437b-925a-4b89d5595dc0"
-					(reference "#PWR097")
-					(unit 1)
-				)
+					(reference "#PWR0106")
+					(unit 1)
+				)

Commit message: more routing
Parts:
- C66, C67, C68, C69: voltage (none) -> 10
Changed lines of the file:
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@@
+			)
+		)
+		(property "voltage" "10"
+			(at 25.4 113.03 0)
+			(effects
+				(font
+					(size 1.27 1.27)
+				)
+				(hide yes)
 			)
 		)
@@
 			)
 		)
+		(property "voltage" "10"
+			(at 63.5 113.03 0)
+			(effects
+				(font
+					(size 1.27 1.27)
+				)
+				(hide yes)
+			)
+		)
 		(pin "1"
 		)
@@
 			)
 		)
+		(property "voltage" "10"
+			(at 38.1 113.03 0)
+			(effects
+				(font
+					(size 1.27 1.27)
+				)
+				(hide yes)
+			)
+		)
 		(pin "1"
 		)
@@
 			(at 50.8 113.03 0)
 			(effects
+				(font
+					(size 1.27 1.27)
+				)
+				(hide yes)
+			)
+		)
+		(property "voltage" "10"
+			(at 50.8 113.03 0)
+			(effects

Commit message: Formatting
Other:
- company: (none) -> UMASS Cubesat Lab
Changed lines of the file:
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@@
 	(generator_version "9.0")
 	(paper "A5")
+	(title_block
+		(date "2026-03-22")
+		(rev "R1")
+		(company "UMASS Cubesat Lab")
+	)
 	(rectangle
 		(start 81.28 59.69)

Commit message: R1 candidate
Connections:
- net +3.3V: now also U11.3 (IO2), U11.7 (IO3), U12.3 (IO2), U12.7 (IO3), U13.3 (IO2), U13.7 (IO3), U14.3 (IO2), U14.7 (IO3)
- no-connect marks 8 -> 0
Other:
- moved on the sheet: U11
