File: QSPI.kicad_sch (KiCad schematic)
At the start: 2 parts, among them U9 W25Q128JVS

Commit message: Finish IMS, finished more work on schematic
Parts:
- C51: renamed from C39; footprint (none) -> Capacitor_SMD:C_0402_1005Metric
- renumbered U9 to U5
Other:
- moved on the sheet: C51, U5

Commit message: Beginnings of routing
Parts:
- renumbered U5 to U6
Changed lines of the file:
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@@
 		(dnp no)
 		(fields_autoplaced yes)
-		(property "Reference" "#PWR068"
+		(property "Reference" "#PWR075"
 			(at 77.47 90.17 0)
 			(effects
@@
 			(project ""
 				(path "/f01d9098-91c1-4e97-a02a-fecce6a76317/df70517b-b72b-42a5-bf6b-49f6072d6722"
-					(reference "#PWR068")
+					(reference "#PWR075")
 					(unit 1)
 				)
@@
 		(on_board yes)
 		(dnp no)
-		(property "Reference" "U5"
+		(property "Reference" "U6"
 			(at 68.58 62.23 0)
 			(effects
@@
 			(project "Cubesat-FC-V1"
 				(path "/f01d9098-91c1-4e97-a02a-fecce6a76317/df70517b-b72b-42a5-bf6b-49f6072d6722"
-					(reference "U5")
+					(reference "U6")
 					(unit 1)
 				)
@@
 		(dnp no)
 		(fields_autoplaced yes)
-		(property "Reference" "#PWR070"
+		(property "Reference" "#PWR073"
 			(at 92.71 54.61 0)
 			(effects
@@
 			(project "Cubesat-FC-V1"
 				(path "/f01d9098-91c1-4e97-a02a-fecce6a76317/df70517b-b72b-42a5-bf6b-49f6072d6722"
-					(reference "#PWR070")
+					(reference "#PWR073")
 					(unit 1)
 				)
@@
 		(dnp no)
 		(fields_autoplaced yes)
-		(property "Reference" "#PWR067"
+		(property "Reference" "#PWR074"
 			(at 77.47 64.77 0)
 			(effects
@@
 			(project ""
 				(path "/f01d9098-91c1-4e97-a02a-fecce6a76317/df70517b-b72b-42a5-bf6b-49f6072d6722"
-					(reference "#PWR067")
+					(reference "#PWR074")
 					(unit 1)
 				)
@@
 		(dnp no)
 		(fields_autoplaced yes)
-		(property "Reference" "#PWR069"
+		(property "Reference" "#PWR072"
 			(at 92.71 44.45 0)
 			(effects
@@
 			(project "Cubesat-FC-V1"
 				(path "/f01d9098-91c1-4e97-a02a-fecce6a76317/df70517b-b72b-42a5-bf6b-49f6072d6722"
-					(reference "#PWR069")
-					(unit 1)
-				)
+					(reference "#PWR072")
+					(unit 1)
+				)

Commit message: more routing
Parts:
- C51: voltage (none) -> 10
Changed lines of the file:
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@@
+			)
+		)
+		(property "voltage" "10"
+			(at 92.71 44.45 0)
+			(effects
+				(font
+					(size 1.27 1.27)
+				)
+				(hide yes)
 			)
 		)

Commit message: Formatting
Other:
- company: (none) -> UMASS Cubesat Lab
Changed lines of the file:
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@@
 	(generator_version "9.0")
 	(paper "A5")
+	(title_block
+		(date "2026-03-22")
+		(rev "R1")
+		(company "UMASS Cubesat Lab")
+	)
 	(bus_entry
 		(at 123.19 45.72)

Commit message: R1 candidate
Changed lines of the file:
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@@
-	(wire
-		(pts
-			(xy 114.3 63.5) (xy 132.08 63.5)
-		)
-		(stroke
-			(width 0)
-			(type default)
-		)
-	)
 	(wire
 		(pts
@@
 		)
 	)
+	(wire
+		(pts
+			(xy 63.5 69.85) (xy 64.77 69.85)
+		)
+		(stroke
+			(width 0)
+			(type default)
+		)
+	)
 	(bus
 		(pts
@@
 		(pts
 			(xy 63.5 74.93) (xy 64.77 74.93)
-		)
-		(stroke
-			(width 0)
-			(type default)
-		)
-	)
-	(wire
-		(pts
-			(xy 41.91 69.85) (xy 64.77 69.85)
 		)
 		(stroke
@@
 		)
 	)
-	(label "QSPI_FLASH0_CS"
-		(at 41.91 69.85 0)
-		(effects
-			(font
-				(size 1.27 1.27)
-			)
-			(justify left bottom)
-		)
-	)
 	(label "QSPI_D2"
 		(at 114.3 43.18 0)
@@
 		)
 	)
-	(label "QSPI_FLASH0_CS"
-		(at 114.3 63.5 0)
-		(effects
-			(font
-				(size 1.27 1.27)
-			)
-			(justify left bottom)
-		)
-	)
 	(label "QSPI_D3"
 		(at 114.3 45.72 0)
@@
 	(hierarchical_label "QSPI_FLASH0_CS"
 		(shape input)
-		(at 132.08 63.5 0)
-		(effects
-			(font
-				(size 1.27 1.27)
-			)
-			(justify left)
-		)
-	)
+		(at 63.5 69.85 180)
+		(effects
+			(font
+				(size 1.27 1.27)
+			)
+			(justify right)
+		)
+	)
