File: STM32H747.kicad_sch (KiCad schematic)
At the start: 46 parts, among them SW1 SW_Button, U3 STM32H757IITx, Y1 ASCO, Y2 32.768KHZ

Commit message: Finish IMS, finished more work on schematic
Parts:
- removed JP1, JP2: Jumper, symbol Jumper:Jumper_3_Open
- removed R1, R2: R_Small, symbol Device:R_Small
- removed SW1: SW_Button, symbol Switch:SW_Omron_B3FS
- removed U3: STM32H757IITx, Package_QFP:LQFP-176_24x24mm_P0.5mm, symbol MCU_ST_STM32H7:STM32H757IITx
- added U3: STM32H757BITx, Package_QFP:LQFP-208_28x28mm_P0.5mm, symbol MCU_ST_STM32H7:STM32H757BITx
- C12: renamed from C1; footprint (none) -> Capacitor_SMD:C_0402_1005Metric
- C13: renamed from C17; footprint (none) -> Capacitor_SMD:C_0402_1005Metric
- C14: renamed from C34; footprint (none) -> Capacitor_SMD:C_0402_1005Metric
- C15: renamed from C16; footprint (none) -> Capacitor_SMD:C_0402_1005Metric
- C16: renamed from C33; footprint (none) -> Capacitor_SMD:C_0402_1005Metric
- C17: renamed from C2; footprint (none) -> Capacitor_SMD:C_0402_1005Metric
- C18: footprint (none) -> Capacitor_SMD:C_0402_1005Metric
- C19: renamed from C24; footprint (none) -> Capacitor_SMD:C_0402_1005Metric
- C20: renamed from C32; footprint (none) -> Capacitor_SMD:C_0402_1005Metric
- C21: renamed from C3; footprint (none) -> Capacitor_SMD:C_0402_1005Metric
- C22: renamed from C19; footprint (none) -> Capacitor_SMD:C_0402_1005Metric
- C23: renamed from C4; footprint (none) -> Capacitor_SMD:C_0402_1005Metric
- C24: renamed from C20; footprint (none) -> Capacitor_SMD:C_0402_1005Metric
- C25: renamed from C5; footprint (none) -> Capacitor_SMD:C_0402_1005Metric
- C26: renamed from C21; footprint (none) -> Capacitor_SMD:C_0402_1005Metric
- C27: renamed from C36; footprint (none) -> Capacitor_SMD:C_0402_1005Metric
- C28: renamed from C30; footprint (none) -> Capacitor_SMD:C_0402_1005Metric
- C29: renamed from C37; footprint (none) -> Capacitor_SMD:C_0402_1005Metric
- C30: renamed from C6; footprint (none) -> Capacitor_SMD:C_0402_1005Metric
- C31: renamed from C22; footprint (none) -> Capacitor_SMD:C_0402_1005Metric
- C32: renamed from C35; footprint (none) -> Capacitor_SMD:C_0402_1005Metric
- C33: renamed from C31; footprint (none) -> Capacitor_SMD:C_0402_1005Metric
- C34: renamed from C7; footprint (none) -> Capacitor_SMD:C_0402_1005Metric
- C35: renamed from C23; footprint (none) -> Capacitor_SMD:C_0402_1005Metric
- C36: renamed from C28; footprint (none) -> Capacitor_SMD:C_0402_1005Metric
- C37: renamed from C8; footprint (none) -> Capacitor_SMD:C_0402_1005Metric
- C38: renamed from C13; footprint (none) -> Capacitor_SMD:C_0402_1005Metric
- C39: renamed from C9; footprint (none) -> Capacitor_SMD:C_0402_1005Metric
- C40: renamed from C14; footprint (none) -> Capacitor_SMD:C_0402_1005Metric
- C41: renamed from C25; footprint (none) -> Capacitor_SMD:C_0402_1005Metric
- C42: renamed from C10; footprint (none) -> Capacitor_SMD:C_0402_1005Metric
- C43: renamed from C15; footprint (none) -> Capacitor_SMD:C_0402_1005Metric
- C44: renamed from C29; footprint (none) -> Capacitor_SMD:C_0402_1005Metric
- C45: renamed from C26; footprint (none) -> Capacitor_SMD:C_0402_1005Metric
- C46: renamed from C11; footprint (none) -> Capacitor_SMD:C_0402_1005Metric
- C47: renamed from C12; footprint (none) -> Capacitor_SMD:C_0402_1005Metric
- C48: renamed from C27; footprint (none) -> Capacitor_SMD:C_0402_1005Metric
- FB1: footprint (none) -> Resistor_SMD:R_0402_1005Metric
- renumbered Y2 to Y1, Y1 to Y2
Connections:
- net +3.3V: now also U3.100 (VDD), U3.108 (VDD), U3.114 (VDD), U3.117 (VDD), U3.133 (VDD), U3.140 (VDD50_USB), U3.141 (VDD33_USB), U3.154 (VDDLDO), U3.155 (VDD), U3.161 (VDD), U3.17 (VDD), U3.179 (VDD), U3.187 (VDD), U3.202 (VDDLDO), U3.208 (VDD), U3.29 (VDD), U3.49 (VDD), U3.56 (VDD), U3.7 (VDD), U3.74 (VDD), U3.8 (VBAT), U3.80 (VDD), U3.91 (VDDLDO)
- net +3.3VA: now also U3.43 (VREF+), U3.44 (VDDA)
- net BOOT0: now also U3.194 (BOOT0)
- net FMCA0: now also U3.22 (PF0)
- net FMCA1: now also U3.23 (PF1)
- net FMCA10: now also U3.72 (PG0)
- net FMCA11: now also U3.75 (PG1)
- net FMCA12: now also U3.130 (PG2)
- net FMCA2: now also U3.24 (PF2)
- net FMCA3: now also U3.25 (PF3)
- net FMCA4: now also U3.26 (PF4)
- net FMCA5: now also U3.27 (PF5)
- net FMCA6: now also U3.68 (PF12)
- net FMCA7: now also U3.69 (PF13)
- net FMCA8: now also U3.70 (PF14)
- net FMCA9: now also U3.71 (PF15)
- net FMCBA0: now also U3.134 (PG4)
- net FMCBA1: now also U3.135 (PG5)
- net FMCD0: now also U3.115 (PD14)
- net FMCD1: now also U3.116 (PD15)
- net FMCD10: now also U3.84 (PE13)
- net FMCD11: now also U3.85 (PE14)
- net FMCD12: now also U3.86 (PE15)
- net FMCD13: now also U3.105 (PD8)
- net FMCD14: now also U3.106 (PD9)
- net FMCD15: now also U3.107 (PD10)
- net FMCD2: now also U3.170 (PD0)
- net FMCD3: now also U3.171 (PD1)
- net FMCD4: now also U3.76 (PE7)
- net FMCD5: now also U3.77 (PE8)
- net FMCD6: now also U3.78 (PE9)
- net FMCD7: now also U3.81 (PE10)
- net FMCD8: now also U3.82 (PE11)
- net FMCD9: now also U3.83 (PE12)
- net FMCNBL0: now also U3.197 (PE0)
- net FMCNBL1: now also U3.198 (PE1)
- net FMCSDCKE0: now also U3.62 (PC5)
- net FMCSDCLK: now also U3.138 (PG8)
- net FMCSDNCAS: now also U3.188 (PG15)
- net FMCSDNE0: now also U3.61 (PC4)
- net FMCSDNRAS: now also U3.67 (PF11)
- net FMCSDNWE: now also U3.60 (PA7)
- net GND: now also U3.109 (VSS), U3.113 (VSS), U3.118 (VSS), U3.123 (VSSDSI), U3.129 (VSSDSI), U3.132 (VSS), U3.139 (VSS), U3.153 (VSS), U3.16 (VSS), U3.160 (VSS), U3.178 (VSS), U3.18 (VSSSMPS), U3.186 (VSS), U3.200 (VSS), U3.207 (VSS), U3.28 (VSS), U3.42 (VSSA), U3.50 (VSS), U3.55 (VSS), U3.6 (VSS), U3.73 (VSS), U3.79 (VSS), U3.90 (VSS), U3.99 (VSS)
- net HFOSC_IN: now also U3.35 (PH0)
- net LFOSC_IN: now also U3.11 (PC14)
- net LFOSC_OUT: now also U3.12 (PC15)
- net NRST: now also U3.37 (NRST)
- net PDR_EN: now also U3.201 (PDR_ON)
- net QSPI_BK1_IO0: now also U3.32 (PF8)
- net QSPI_BK1_IO1: now also U3.33 (PF9)
- net QSPI_BK1_IO2: now also U3.31 (PF7)
- net QSPI_BK1_IO3: now also U3.30 (PF6)
- net QSPI_BK1_NCS: now also U3.87 (PB10)
- net QSPI_CLK: now also U3.34 (PF10)
- net SWD_TCK/SWCLK: now also U3.165 (PA14)
- net SWD_TDI: now also U3.166 (PA15)
- net SWD_TDO/SWO: now also U3.189 (PB3)
- net SWD_TMS/SWDIO: now also U3.151 (PA13)
- net SWD_TRACE_CK: now also U3.1 (PE2)
- net SWD_TRACE_D0: now also U3.2 (PE3)
- net SWD_TRACE_D1: now also U3.3 (PE4)
- net SWD_TRACE_D2: now also U3.4 (PE5)
- net SWD_TRACE_D3: now also U3.5 (PE6)
- net SWD_TRST: now also U3.190 (PB4)
- net VCAP: now also U3.152 (VCAP), U3.199 (VCAP), U3.89 (VCAP)
- net VCAPDSI: now also U3.119 (VCAPDSI), U3.120 (VDD12DSI), U3.126 (VDD12DSI)
- new net CS_INS_IMU_PRI: U3.38 (PC0)
- new net CS_INS_IMU_SEC0: U3.39 (PC1)
- new net CS_INS_IMU_SEC1: U3.40 (PC2_C)
- new net CS_INS_MAG: U3.41 (PC3_C)
- new net CS_STORAGE_CATALOG0: U3.146 (PA8)
- new net CS_STORAGE_CATALOG1: U3.147 (PA9)
- new net CS_STORAGE_CATALOG2: U3.148 (PA10)
- new net CS_STORAGE_DATALOG: U3.58 (PA5)
- new net CUR_MEAS: U3.63 (PB0)
- new net DCMID0: U3.95 (PH9)
- new net DCMID1: U3.96 (PH10)
- new net DCMID10: U3.164 (PI3)
- new net DCMID11: U3.158 (PH15)
- new net DCMID12: U3.136 (PG6)
- new net DCMID13: U3.137 (PG7)
- new net DCMID2: U3.97 (PH11)
- new net DCMID3: U3.98 (PH12)
- new net DCMID4: U3.157 (PH14)
- new net DCMID5: U3.203 (PI4)
- new net DCMID6: U3.205 (PI6)
- new net DCMID7: U3.206 (PI7)
- new net DCMID8: U3.162 (PI1)
- new net DCMID9: U3.163 (PI2)
- new net DCMI_HSYNC: U3.57 (PA4)
- new net DCMI_PIXCLK: U3.59 (PA6)
- new net DCMI_VSYNC: U3.204 (PI5)
- new net FDCAN1_RX/UART4_RX: U3.195 (PB8)
- new net FDCAN1_TX/UART4_TX: U3.196 (PB9)
- new net FDCAN2_RX: U3.191 (PB5)
- new net FDCAN2_TX: U3.192 (PB6)
- new net I2C2_SCL: U3.52 (PH4)
- new net I2C2_SDA: U3.53 (PH5)
- new net INT_IMU_PRI_DRDY: U3.173 (PD3)
- new net PIN_BUZZER: U3.92 (PH6)
- new net PIN_CONFIG_0: U3.15 (PI11)
- new net PIN_CONFIG_1: U3.66 (PI15)
- new net PIN_CONFIG_2: U3.36 (PH1)
- new net PIN_CONFIG_3: U3.48 (PH2)
- new net PIN_GPIO_PWM0: U3.64 (PB1)
- new net PIN_GPIO_PWM1: U3.65 (PB2)
- new net PIN_PROC0BUSY: U3.9 (PI8)
- new net PIN_PROC0GP0: U3.13 (PI9)
- new net PIN_PROC0GP1: U3.14 (PI10)
- new net PIN_PROC1BUSY: U3.110 (PD11)
- new net PIN_PROC1GP0: U3.111 (PD12)
- new net PIN_PROC1GP1: U3.112 (PD13)
- new net SDMMC1_CK: U3.169 (PC12)
- new net SDMMC1_CMD: U3.172 (PD2)
- new net SDMMC1_D0: U3.144 (PC8)
- new net SDMMC1_D0DIR: U3.142 (PC6)
- new net SDMMC1_D1: U3.145 (PC9)
- new net SDMMC1_D123DIR: U3.143 (PC7)
- new net SDMMC1_D2: U3.167 (PC10)
- new net SDMMC1_D3: U3.168 (PC11)
- new net SPI1_CIPO: U3.180 (PG9)
- new net SPI1_COPI: U3.183 (PG12)
- new net SPI1_SCK: U3.182 (PG11)
- new net SPI2_CIPO: U3.103 (PB14)
- new net SPI2_COPI: U3.104 (PB15)
- new net SPI2_SCK: U3.102 (PB13)
- new net USART2_RX: U3.176 (PD6)
- new net USART2_TX: U3.175 (PD5)
- new net USB_FS_DM: U3.150 (PA12)
- new net USB_FS_DP: U3.149 (PA11)
- no-connect marks 8 -> 9
Other:
- note added: "Double check that DP/DM are the only pins needed for USB FS"
- note added: "Reset button"
- note removed: "Power supervision system enable"
- note removed: "Reset and configuration"
- note removed: "boot mode selection"
- moved on the sheet: C14, C15, C16, C19, C27, C28, C32, C33, C44, FB1, Y1, Y2

Commit message: Beginnings of routing
Parts:
- Y1: footprint (none) -> Crystal:Crystal_SMD_Abracon_ABM3-2Pin_5.0x3.2mm
- renumbered C17 to C13, C21 to C14, C23 to C15, C25 to C16, C30 to C17, C34 to C18, C37 to C19, C39 to C20, C42 to C21, C46 to C22, C13 to C23, C18 to C24, C22 to C25, C24 to C26, C26 to C27, C31 to C28, C35 to C29, C38 to C30, C40 to C31, C43 to C32, C47 to C33, C44 to C34, C15 to C35, C19 to C36, C28 to C37, C33 to C38, C20 to C39, C29 to C40, C36 to C41, C41 to C42, C45 to C43, C48 to C44, C27 to C45, C32 to C46, C14 to C47, C16 to C48, U3 to U4
Connections:
- net CS_STORAGE_CATALOG0: now also U4.181 (PG10); no longer U4.146 (PA8)
- net CS_STORAGE_CATALOG1: now also U4.184 (PG13); no longer U4.147 (PA9)
- net CS_STORAGE_CATALOG2: now also U4.185 (PG14); no longer U4.148 (PA10)
- net CS_STORAGE_DATALOG: now also U4.177 (PD7); no longer U4.58 (PA5)
- net PIN_CONFIG_2: now also U4.48 (PH2); no longer U4.36 (PH1)
- net PIN_CONFIG_3: now also U4.51 (PH3); no longer U4.48 (PH2)
- net UART4_TX: now reaches U4.45 (PA0)
- net UART4_RX: now reaches U4.46 (PA1)
- net I2C3_SCL: now reaches U4.93 (PH7)
- net I2C3_SDA: now reaches U4.94 (PH8)
- net FDCAN1_RX/UART4_RX renamed FDCAN1_RX
- net FDCAN1_TX/UART4_TX renamed FDCAN1_TX
- new net USB_FS_VBUS: U4.147 (PA9)

Commit message: more routing
Parts:
- C12, C13, C14, C15, C16, C17, C18, C19, C20, C21, C22, C23, C24, C25, C26, C27, C28, C29, C30, C31, C32, C33, C34, C35, C36, C37, C38, C39, C40, C41, C42, C43, C44, C45, C46, C47, C48: voltage (none) -> 10
Connections:
- net GND: now also C16.2

Commit message: more routing
Connections:
- net CS_INS_IMU_SEC1: now also U4.41 (PC3_C); no longer U4.40 (PC2_C)
- net CS_INS_MAG: now also U4.40 (PC2_C); no longer U4.41 (PC3_C)

Commit message: Formatting
Connections:
- no-connect marks 9 -> 23
Other:
- company: (none) -> UMASS Cubesat Lab
- title: (none) -> STM32H7 Microcontroller
- moved on the sheet: C39, C40, C41, C42, C43, C44, C45, C46, C47, C48, Y1, Y2

Commit message: R1 candidate
Parts:
- C47, C48: value ?? -> 15p
- FB1: value ??? -> 600ohm@1mhz
- Y2: value ASCO -> 24MHZ
Connections:
- removed net VCAP: C42.1, C43.1, C44.1, U4.152 (VCAP), U4.199 (VCAP), U4.89 (VCAP)
- new net VCAP0: C42.1, U4.89 (VCAP)
- new net VCAP1: C43.1, U4.152 (VCAP)
- new net VCAP2: C44.1, U4.199 (VCAP)
Other:
- note removed: "It is unclear if a third VCAP capacitor is needed"
Changed lines of the file:
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@@
 		)
 	)
-	(text "It is unclear if a third \nVCAP capacitor is needed"
-		(exclude_from_sim no)
-		(at 370.332 117.856 0)
-		(effects
-			(font
-				(size 1.27 1.27)
-			)
-			(justify left)
-		)
-	)
 	(text "Note on SMPS:\nThe SMPS uses a switching voltage regulator to increase \nthe efficiency of the STM32, but given the added complexity \nand relatively small gain in power efficiency (plus the \nrisk of the switching FETs latching in space), I dont think \nthis is necesarry."
 		(exclude_from_sim no)
@@
 	)
 	(junction
-		(at 100.33 256.54)
-		(diameter 0)
-		(color 0 0 0 0)
-	)
-	(junction
 		(at 302.26 62.23)
 		(diameter 0)
@@
 	)
 	(junction
-		(at 378.46 120.65)
-		(diameter 0)
-		(color 0 0 0 0)
-	)
-	(junction
 		(at 364.49 54.61)
 		(diameter 0)
@@
 	)
 	(junction
-		(at 100.33 254)
-		(diameter 0)
-		(color 0 0 0 0)
-	)
-	(junction
 		(at 320.04 54.61)
 		(diameter 0)
@@
 	)
 	(junction
-		(at 369.57 120.65)
-		(diameter 0)
-		(color 0 0 0 0)
-	)
-	(junction
 		(at 127 31.75)
 		(diameter 0)
@@
 	(wire
 		(pts
-			(xy 378.46 120.65) (xy 387.35 120.65)
-		)
-		(stroke
-			(width 0)
-			(type default)
-		)
-	)
-	(wire
-		(pts
 			(xy 340.36 91.44) (xy 340.36 92.71)
 		)
@@
 	(wire
 		(pts
-			(xy 100.33 254) (xy 100.33 256.54)
-		)
-		(stroke
-			(width 0)
-			(type default)
-		)
-	)
-	(wire
-		(pts
 			(xy 373.38 29.21) (xy 382.27 29.21)
 		)
@@
 	(wire
 		(pts
-			(xy 369.57 120.65) (xy 378.46 120.65)
-		)
-		(stroke
-			(width 0)
-			(type default)
-		)
-	)
-	(wire
-		(pts
 			(xy 363.22 156.21) (xy 373.38 156.21)
 		)
@@
 	(wire
 		(pts
+			(xy 382.27 120.65) (xy 387.35 120.65)
+		)
+		(stroke
+			(width 0)
+			(type default)
+		)
+	)
+	(wire
+		(pts
 			(xy 373.38 86.36) (xy 373.38 90.17)
 		)
@@
 	(wire
 		(pts
-			(xy 101.6 254) (xy 100.33 254)
-		)
-		(stroke
-			(width 0)
-			(type default)
-		)
-	)
-	(wire
-		(pts
 			(xy 203.2 78.74) (xy 204.47 78.74)
 		)
@@
 	(wire
 		(pts
+			(xy 88.9 251.46) (xy 101.6 251.46)
+		)
+		(stroke
+			(width 0)
+			(type default)
+		)
+	)
+	(wire
+		(pts
 			(xy 203.2 172.72) (xy 212.09 172.72)
 		)
@@
 	(wire
 		(pts
+			(xy 88.9 256.54) (xy 101.6 256.54)
+		)
+		(stroke
+			(width 0)
+			(type default)
+		)
+	)
+	(wire
+		(pts
 			(xy 182.88 31.75) (xy 182.88 33.02)
 		)
@@
 	(wire
 		(pts
-			(xy 101.6 251.46) (xy 100.33 251.46)
-		)
-		(stroke
-			(width 0)
-			(type default)
-		)
-	)
-	(wire
-		(pts
 			(xy 203.2 210.82) (xy 212.09 210.82)
 		)
@@
 	(wire
 		(pts
+			(xy 373.38 120.65) (xy 378.46 120.65)
+		)
+		(stroke
+			(width 0)
+			(type default)
+		)
+	)
+	(wire
+		(pts
 			(xy 100.33 134.62) (xy 101.6 134.62)
 		)
@@
 	(wire
 		(pts
+			(xy 88.9 254) (xy 101.6 254)
+		)
+		(stroke
+			(width 0)
+			(type default)
+		)
+	)
+	(wire
+		(pts
 			(xy 382.27 60.96) (xy 382.27 62.23)
 		)
@@
 	(wire
 		(pts
-			(xy 100.33 251.46) (xy 100.33 254)
-		)
-		(stroke
-			(width 0)
-			(type default)
-		)
-	)
-	(wire
-		(pts
 			(xy 364.49 62.23) (xy 373.38 62.23)
 		)
@@
 	(wire
 		(pts
-			(xy 88.9 256.54) (xy 100.33 256.54)
-		)
-		(stroke
-			(width 0)
-			(type default)
-		)
-	)
-	(wire
-		(pts
 			(xy 100.33 60.96) (xy 101.6 60.96)
 		)
@@
 	(wire
 		(pts
-			(xy 100.33 256.54) (xy 101.6 256.54)
-		)
-		(stroke
-			(width 0)
-			(type default)
-		)
-	)
-	(wire
-		(pts
 			(xy 320.04 30.48) (xy 320.04 29.21)
 		)
@@
 		)
 	)
+	(label "VCAP1"
+		(at 373.38 120.65 0)
+		(effects
+			(font
+				(size 1.27 1.27)
+			)
+			(justify left bottom)
+		)
+	)
 	(label "FMCA1"
 		(at 88.9 210.82 0)
@@
 		)
 	)
+	(label "VCAP2"
+		(at 88.9 256.54 0)
+		(effects
+			(font
+				(size 1.27 1.27)
+			)
+			(justify left bottom)
+		)
+	)
 	(label "FMCD15"
 		(at 234.95 198.12 180)
@@
 		)
 	)
+	(label "VCAP0"
+		(at 364.49 120.65 0)
+		(effects
+			(font
+				(size 1.27 1.27)
+			)
+			(justify left bottom)
+		)
+	)
 	(label "FMCA5"
 		(at 88.9 220.98 0)
@@
 		)
 	)
-	(label "VCAP"
-		(at 88.9 256.54 0)
+	(label "VCAP0"
+		(at 88.9 251.46 0)
 		(effects
 			(font
@@
 		)
 	)
-	(label "VCAP"
-		(at 364.49 120.65 0)
+	(label "VCAP2"
+		(at 382.27 120.65 0)
 		(effects
 			(font
@@
 		)
 	)
+	(label "VCAP1"
+		(at 88.9 254 0)
+		(effects
+			(font
+				(size 1.27 1.27)
+			)
+			(justify left bottom)
+		)
+	)
 	(label "FMCA6"
 		(at 80.01 238.76 0)
@@
 			)
 		)
-		(property "Value" "??"
+		(property "Value" "15p"
 			(at 302.26 158.7562 0)
 			(effects
@@
 			)
 		)
-		(property "Value" "???"
+		(property "Value" "600ohm@1mhz"
 			(at 314.9219 87.63 90)
 			(effects
@@
 			)
 		)
-		(property "Value" "??"
+		(property "Value" "15p"
 			(at 292.1 158.7562 0)
 			(effects
@@
 		(fields_autoplaced yes)
 		(property "Reference" "Y2"
-			(at 364.49 149.7898 0)
+			(at 365.76 149.7898 0)
 			(effects
 				(font
@@
 			)
 		)
-		(property "Value" "ASCO"
-			(at 364.49 152.3298 0)
+		(property "Value" "24MHZ"
+			(at 365.76 152.3298 0)
 			(effects
 				(font
